Commit message: Update stp and urdf files of esrobo to adapt to officially given urdf files

File: model/urdf/esrobo_waist_with_head/urdf/esrobo_waist_with_head.urdf (robot description, URDF)
Before this commit: robot esrobo_waist_with_head, 10 links, 9 joints
Links:
- added link leftSensor_link, mass 0.254777372478428; collision mesh filename=package://esrobo_waist_with_head/meshes/leftSensor_link.STL; visual mesh filename=package://esrobo_waist_with_head/meshes/leftSensor_link.STL
- added link rightSensor_link, mass 0.238356407740794; collision mesh filename=package://esrobo_waist_with_head/meshes/rightSensor_link.STL; visual mesh filename=package://esrobo_waist_with_head/meshes/rightSensor_link.STL
- link head_link2: mass 0.256259573814006 -> 0.256259573813189
- link leftArm_link: mass 0.900253820886967 -> 0.900253813427799
- link rightArm_link: mass 0.900257859569218 -> 0.900257809789524
- link waist_base: mass 1.29464248262156 -> 1.2946424823519
- link waist_link1: mass 2.61616405831954 -> 2.6161640614807
- link waist_link2: mass 2.01092959064243 -> 2.01092959225819
- link waist_link3: mass 7.46035492035243 -> 7.46035263489036
Joints:
- added joint leftSensor_joint: type fixed, parent leftArm_link, child leftSensor_link, origin xyz=-0.0012639 -0.613 -0.1381 rpy=0 0 0, axis 0 0 0
- added joint rightSensor_joint: type fixed, parent rightArm_link, child rightSensor_link, origin xyz=-0.0017158 -0.613 0.1381 rpy=0 0 0, axis 0 0 0
- joint head_joint1: limit lower=-1.57 upper=1.57 effort=0 velocity=0 -> lower=0 upper=6.28 effort=0 velocity=0
- joint leftArm_joint: limit lower=0 upper=1.57 effort=0 velocity=0 -> lower=0 upper=3.14 effort=0 velocity=0; origin xyz=0.0078413 0.42849 -0.1744 rpy=0 0 0 -> xyz=0.0076949 0.42752 -0.086398 rpy=0 0 0
- joint rightArm_joint: limit lower=0 upper=1.57 effort=0 velocity=0 -> lower=0 upper=3.14 effort=0 velocity=0; origin xyz=0.0072359 0.42849 0.1956 rpy=0 0 0 -> xyz=0.0073775 0.42752 0.1076 rpy=0 0 0
- joint waist_baseJoint: origin xyz=-0.156416685832191 0 0 rpy=1.5707963267949 0 0 -> xyz=-0.15642 0 0 rpy=1.5708 0 0

Commit message: Add hand base coordinate system

File: model/urdf/esrobo_waist_with_head/urdf/esrobo_waist_with_head.urdf (robot description, URDF)
Before this commit: robot esrobo_waist_with_head, 12 links, 11 joints
Links:
- added link leftHand_link, mass 0.307600132223361; collision mesh filename=package://esrobo_waist_with_head/meshes/leftHand_link.STL; visual mesh filename=package://esrobo_waist_with_head/meshes/leftHand_link.STL
- added link rightHand_link, mass 0.307600134187615; collision mesh filename=package://esrobo_waist_with_head/meshes/rightHand_link.STL; visual mesh filename=package://esrobo_waist_with_head/meshes/rightHand_link.STL
- link base_link: mass 21.7638613943257 -> 21.7638613943256
- link head_link2: mass 0.256259573813189 -> 0.256259570812732
- link leftArm_link: mass 0.900253813427799 -> 0.900253820880401
- link rightArm_link: mass 0.900257809789524 -> 0.900257901077131
- link waist_base: mass 1.2946424823519 -> 1.2946424823513
- link waist_link1: mass 2.6161640614807 -> 2.61616445921771
- link waist_link3: mass 7.46035263489036 -> 7.46035263489037
Joints:
- added joint leftHand_joint: type fixed, parent leftSensor_link, child leftHand_link, origin xyz=-0.00021023 -0.0865 0 rpy=0 0 0, axis 0 0 0
- added joint rightHand_joint: type fixed, parent rightSensor_link, child rightHand_link, origin xyz=-0.00021023 -0.0865 0 rpy=0 0 0, axis 0 0 0
- joint lidar_joint: origin xyz=0.299141092446627 -0.00804855452219633 0 rpy=0 0 0 -> xyz=0.29914 -0.0080486 0 rpy=0 0 0
