Commit message: Integrate officially provided urdf files of arm and hand with the raw urdf file exported by sw

File: model/urdf/esrobo_waist_with_head/urdf/esrobo_waist_with_head.urdf (robot description, URDF)
Before this commit: robot esrobo_waist_with_head, 14 links, 13 joints
Links:
- added link left_index_distal, mass 0.0031445375098231; collision mesh filename=package://esrobo_waist_with_head/meshes/linkerhand_l20lite/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; visual mesh filename=package://esrobo_waist_with_head/meshes/linkerhand_l20lite/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
- added link left_index_metacarpals, mass 0.0038877126435198; collision mesh filename=package://esrobo_waist_with_head/meshes/linkerhand_l20lite/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; visual mesh filename=package://esrobo_waist_with_head/meshes/linkerhand_l20lite/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
- added link left_index_middle, mass 0.00283043921422803; collision mesh filename=package://esrobo_waist_with_head/meshes/linkerhand_l20lite/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; visual mesh filename=package://esrobo_waist_with_head/meshes/linkerhand_l20lite/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
- added link left_index_proximal, mass 0.00316246584579941; collision mesh filename=package://esrobo_waist_with_head/meshes/linkerhand_l20lite/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; visual mesh filename=package://esrobo_waist_with_head/meshes/linkerhand_l20lite/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
- added link left_middle_distal, mass 0.00314452092964384; collision mesh filename=package://esrobo_waist_with_head/meshes/linkerhand_l20lite/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; visual mesh filename=package://esrobo_waist_with_head/meshes/linkerhand_l20lite/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
- added link left_middle_middle, mass 0.00283043921858529; collision mesh filename=package://esrobo_waist_with_head/meshes/linkerhand_l20lite/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; visual mesh filename=package://esrobo_waist_with_head/meshes/linkerhand_l20lite/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
- added link left_middle_proximal, mass 0.00316246719662224; collision mesh filename=package://esrobo_waist_with_head/meshes/linkerhand_l20lite/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; visual mesh filename=package://esrobo_waist_with_head/meshes/linkerhand_l20lite/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
- added link left_nero_base_link, mass 1.06458435; collision mesh filename=package://esrobo_waist_with_head/meshes/nero/base_link.stl; visual mesh filename=package://esrobo_waist_with_head/meshes/nero/dae/base_link.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
- added link left_nero_gripper_flange, mass 0.04771096; collision mesh filename=package://esrobo_waist_with_head/meshes/nero/gripper_flange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; visual mesh filename=package://esrobo_waist_with_head/meshes/nero/dae/gripper_fl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
- added link left_nero_link1, mass 0.76710504; collision mesh filename=package://esrobo_waist_with_head/meshes/nero/link1.stl; visual mesh filename=package://esrobo_waist_with_head/meshes/nero/dae/link1.dae
- added link left_nero_link2, mass 0.69381908; collision mesh filename=package://esrobo_waist_with_head/meshes/nero/link2.stl; visual mesh filename=package://esrobo_waist_with_head/meshes/nero/dae/link2.dae
- added link left_nero_link3, mass 0.67246544; collision mesh filename=package://esrobo_waist_with_head/meshes/nero/link3.stl; visual mesh filename=package://esrobo_waist_with_head/meshes/nero/dae/link3.dae
- added link left_nero_link4, mass 0.48451414; collision mesh filename=package://esrobo_waist_with_head/meshes/nero/link4.stl; visual mesh filename=package://esrobo_waist_with_head/meshes/nero/dae/link4.dae
- added link left_nero_link5, mass 0.58368405; collision mesh filename=package://esrobo_waist_with_head/meshes/nero/link5.stl; visual mesh filename=package://esrobo_waist_with_head/meshes/nero/dae/link5.dae
- added link left_nero_link6, mass 0.3140406; collision mesh filename=package://esrobo_waist_with_head/meshes/nero/link6.stl; visual mesh filename=package://esrobo_waist_with_head/meshes/nero/dae/link6.dae
- added link left_nero_link7, mass 0.000001; collision mesh filename=package://esrobo_waist_with_head/meshes/nero/link7.stl; visual mesh filename=package://esrobo_waist_with_head/meshes/nero/dae/link7.dae
- added link left_pinky_distal, mass 0.00314455887032079; collision mesh filename=package://esrobo_waist_with_head/meshes/linkerhand_l20lite/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; visual mesh filename=package://esrobo_waist_with_head/meshes/linkerhand_l20lite/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
- added link left_pinky_metacarpals, mass 0.00388771229554929; collision mesh filename=package://esrobo_waist_with_head/meshes/linkerhand_l20lite/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; visual mesh filename=package://esrobo_waist_with_head/meshes/linkerhand_l20lite/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
- added link left_pinky_middle, mass 0.00283043906989622; collision mesh filename=package://esrobo_waist_with_head/meshes/linkerhand_l20lite/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; visual mesh filename=package://esrobo_waist_with_head/meshes/linkerhand_l20lite/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
- added link left_pinky_proximal, mass 0.00316246781629033; collision mesh filename=package://esrobo_waist_with_head/meshes/linkerhand_l20lite/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; visual mesh filename=package://esrobo_waist_with_head/meshes/linkerhand_l20lite/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
- added link left_ring_distal, mass 0.00314454943731604; collision mesh filename=package://esrobo_waist_with_head/meshes/linkerhand_l20lite/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; visual mesh filename=package://esrobo_waist_with_head/meshes/linkerhand_l20lite/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
- added link left_ring_metacarpals, mass 0.00388771255966599; collision mesh filename=package://esrobo_waist_with_head/meshes/linkerhand_l20lite/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; visual mesh filename=package://esrobo_waist_with_head/meshes/linkerhand_l20lite/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
- added link left_ring_middle, mass 0.00283043920090097; collision mesh filename=package://esrobo_waist_with_head/meshes/linkerhand_l20lite/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; visual mesh filename=package://esrobo_waist_with_head/meshes/linkerhand_l20lite/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
- added link left_ring_proximal, mass 0.00316246660225829; collision mesh filename=package://esrobo_waist_with_head/meshes/linkerhand_l20lite/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; visual mesh filename=package://esrobo_waist_with_head/meshes/linkerhand_l20lite/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
- added link left_thumb_distal, mass 0.00512798334000111; collision mesh filename=package://esrobo_waist_with_head/meshes/linkerhand_l20lite/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; visual mesh filename=package://esrobo_waist_with_head/meshes/linkerhand_l20lite/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
- added link left_thumb_metacarpals, mass 0.0152011788694593; collision mesh filename=package://esrobo_waist_with_head/meshes/linkerhand_l20lite/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; visual mesh filename=package://esrobo_waist_with_head/meshes/linkerhand_l20lite/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
- added link left_thumb_metacarpals_base1, mass 0.00840514828448049; collision mesh filename=package://esrobo_waist_with_head/meshes/linkerhand_l20lite/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; visual mesh filename=package://esrobo_waist_with_head/meshes/linkerhand_l20lite/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
- added link left_thumb_metacarpals_base2, mass 0.00244725656099355; collision mesh filename=package://esrobo_waist_with_head/meshes/linkerhand_l20lite/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; visual mesh filename=package://esrobo_waist_with_head/meshes/linkerhand_l20lite/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
- added link left_thumb_proximal, mass 0.00662225085289633; collision mesh filename=package://esrobo_waist_with_head/meshes/linkerhand_l20lite/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; visual mesh filename=package://esrobo_waist_with_head/meshes/linkerhand_l20lite/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
- added link right_index_distal, mass 0.0031446130611452; collision mesh filename=package://esrobo_waist_with_head/meshes/linkerhand_l20lite/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; visual mesh filename=package://esrobo_waist_with_head/meshes/linkerhand_l20lite/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
- added link right_index_metacarpals, mass 0.00903700329493157; collision mesh filename=package://esrobo_waist_with_head/meshes/linkerhand_l20lite/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; visual mesh filename=package://esrobo_waist_with_head/meshes/linkerhand_l20lite/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
- added link right_index_middle, mass 0.00283043630937165; collision mesh filename=package://esrobo_waist_with_head/meshes/linkerhand_l20lite/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; visual mesh filename=package://esrobo_waist_with_head/meshes/linkerhand_l20lite/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
- added link right_index_proximal, mass 0.00654982235507964; collision mesh filename=package://esrobo_waist_with_head/meshes/linkerhand_l20lite/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; visual mesh filename=package://esrobo_waist_with_head/meshes/linkerhand_l20lite/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
- added link right_middle_distal, mass 0.00314458659113992; collision mesh filename=package://esrobo_waist_with_head/meshes/linkerhand_l20lite/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; visual mesh filename=package://esrobo_waist_with_head/meshes/linkerhand_l20lite/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
- added link right_middle_middle, mass 0.00283043635504842; collision mesh filename=package://esrobo_waist_with_head/meshes/linkerhand_l20lite/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; visual mesh filename=package://esrobo_waist_with_head/meshes/linkerhand_l20lite/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
- added link right_middle_proximal, mass 0.00654982478226949; collision mesh filename=package://esrobo_waist_with_head/meshes/linkerhand_l20lite/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; visual mesh filename=package://esrobo_waist_with_head/meshes/linkerhand_l20lite/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
- added link right_nero_base_link, mass 1.06458435; collision mesh filename=package://esrobo_waist_with_head/meshes/nero/base_link.stl; visual mesh filename=package://esrobo_waist_with_head/meshes/nero/dae/base_link.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
- added link right_nero_gripper_flange, mass 0.04771096; collision mesh filename=package://esrobo_waist_with_head/meshes/nero/gripper_flange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; visual mesh filename=package://esrobo_waist_with_head/meshes/nero/dae/gripper_fl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
- added link right_nero_link1, mass 0.76710504; collision mesh filename=package://esrobo_waist_with_head/meshes/nero/link1.stl; visual mesh filename=package://esrobo_waist_with_head/meshes/nero/dae/link1.dae
- added link right_nero_link2, mass 0.69381908; collision mesh filename=package://esrobo_waist_with_head/meshes/nero/link2.stl; visual mesh filename=package://esrobo_waist_with_head/meshes/nero/dae/link2.dae
- added link right_nero_link3, mass 0.67246544; collision mesh filename=package://esrobo_waist_with_head/meshes/nero/link3.stl; visual mesh filename=package://esrobo_waist_with_head/meshes/nero/dae/link3.dae
- added link right_nero_link4, mass 0.48451414; collision mesh filename=package://esrobo_waist_with_head/meshes/nero/link4.stl; visual mesh filename=package://esrobo_waist_with_head/meshes/nero/dae/link4.dae
- added link right_nero_link5, mass 0.58368405; collision mesh filename=package://esrobo_waist_with_head/meshes/nero/link5.stl; visual mesh filename=package://esrobo_waist_with_head/meshes/nero/dae/link5.dae
- added link right_nero_link6, mass 0.3140406; collision mesh filename=package://esrobo_waist_with_head/meshes/nero/link6.stl; visual mesh filename=package://esrobo_waist_with_head/meshes/nero/dae/link6.dae
- added link right_nero_link7, mass 0.000001; collision mesh filename=package://esrobo_waist_with_head/meshes/nero/link7.stl; visual mesh filename=package://esrobo_waist_with_head/meshes/nero/dae/link7.dae
- added link right_pinky_distal, mass 0.00314457409502053; collision mesh filename=package://esrobo_waist_with_head/meshes/linkerhand_l20lite/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; visual mesh filename=package://esrobo_waist_with_head/meshes/linkerhand_l20lite/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
- added link right_pinky_metacarpals, mass 0.00903700307878998; collision mesh filename=package://esrobo_waist_with_head/meshes/linkerhand_l20lite/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; visual mesh filename=package://esrobo_waist_with_head/meshes/linkerhand_l20lite/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
- added link right_pinky_middle, mass 0.00283043670305552; collision mesh filename=package://esrobo_waist_with_head/meshes/linkerhand_l20lite/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; visual mesh filename=package://esrobo_waist_with_head/meshes/linkerhand_l20lite/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
- added link right_pinky_proximal, mass 0.00654983474179372; collision mesh filename=package://esrobo_waist_with_head/meshes/linkerhand_l20lite/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; visual mesh filename=package://esrobo_waist_with_head/meshes/linkerhand_l20lite/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
- added link right_ring_distal, mass 0.00314460631735109; collision mesh filename=package://esrobo_waist_with_head/meshes/linkerhand_l20lite/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; visual mesh filename=package://esrobo_waist_with_head/meshes/linkerhand_l20lite/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
- added link right_ring_metacarpals, mass 0.00903700335356623; collision mesh filename=package://esrobo_waist_with_head/meshes/linkerhand_l20lite/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; visual mesh filename=package://esrobo_waist_with_head/meshes/linkerhand_l20lite/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
- added link right_ring_middle, mass 0.0028304363455826; collision mesh filename=package://esrobo_waist_with_head/meshes/linkerhand_l20lite/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; visual mesh filename=package://esrobo_waist_with_head/meshes/linkerhand_l20lite/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
- added link right_ring_proximal, mass 0.00654983629670871; collision mesh filename=package://esrobo_waist_with_head/meshes/linkerhand_l20lite/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; visual mesh filename=package://esrobo_waist_with_head/meshes/linkerhand_l20lite/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
- added link right_thumb_distal, mass 0.00512919991432349; collision mesh filename=package://esrobo_waist_with_head/meshes/linkerhand_l20lite/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; visual mesh filename=package://esrobo_waist_with_head/meshes/linkerhand_l20lite/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
- added link right_thumb_metacarpals, mass 0.0152012256765109; collision mesh filename=package://esrobo_waist_with_head/meshes/linkerhand_l20lite/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; visual mesh filename=package://esrobo_waist_with_head/meshes/linkerhand_l20lite/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
- added link right_thumb_metacarpals_base1, mass 0.0084581547726202; collision mesh filename=package://esrobo_waist_with_head/meshes/linkerhand_l20lite/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; visual mesh filename=package://esrobo_waist_with_head/meshes/linkerhand_l20lite/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
- added link right_thumb_metacarpals_base2, mass 0.00582711245702963; collision mesh filename=package://esrobo_waist_with_head/meshes/linkerhand_l20lite/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; visual mesh filename=package://esrobo_waist_with_head/meshes/linkerhand_l20lite/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
- added link right_thumb_proximal, mass 0.00662231923284161; collision mesh filename=package://esrobo_waist_with_head/meshes/linkerhand_l20lite/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; visual mesh filename=package://esrobo_waist_with_head/meshes/linkerhand_l20lite/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
- link leftArm_link: mass 0.900253820880401 -> None; geometry 
- link leftHand_link: mass 0.307600132223361 -> 0.103652479414672; geometry collision mesh filename=package://esrobo_waist_with_head/meshes/linkerhand_l20lite/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; visual mesh filename=package://esrobo_waist_with_head/meshes/linkerhand_l20lite/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
- link rightArm_link: mass 0.900257901077131 -> None; geometry 
- link rightHand_link: mass 0.307600134187615 -> 0.108844276105116; geometry collision mesh filename=package://esrobo_waist_with_head/meshes/linkerhand_l20lite/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; visual mesh filename=package://esrobo_waist_with_head/meshes/linkerhand_l20lite/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
Joints:
- added joint leftArm_base_joint: type fixed, parent waist_link3, child leftArm_link, origin xyz=0.0075362 0.42752 -0.096999 rpy=0 0 0
- added joint left_index_dip: type revolute, parent left_index_middle, child left_index_distal, origin xyz=-0.0052444 0 0.025711 rpy=0 0 0, axis 0 1 0, limit lower=0 upper=0.62 effort=10.43 velocity=1, mimic joint=left_index_mcp_pitch multiplier=0.46 offset=0
- added joint left_index_mcp_pitch: type revolute, parent left_index_metacarpals, child left_index_proximal, origin xyz=0.0022097 0 0.015275 rpy=0 0 0.00024367, axis 0 1 0, limit lower=0 upper=1.36 effort=4.8 velocity=1
- added joint left_index_mcp_roll: type revolute, parent leftHand_link, child left_index_metacarpals, origin xyz=-0.0021643 -0.026654 0.13253 rpy=0.027927 -0.0087198 -0.00024358, axis 1 0.00024367 0, limit lower=0 upper=0.19 effort=4.29 velocity=1
- added joint left_index_pip: type revolute, parent left_index_proximal, child left_index_middle, origin xyz=-0.0010697 0 0.035634 rpy=0 0 0, axis 0 1 0, limit lower=0 upper=1.78 effort=3.7 velocity=1, mimic joint=left_index_mcp_pitch multiplier=1.3 offset=0
- added joint left_middle_dip: type revolute, parent left_middle_middle, child left_middle_distal, origin xyz=-0.0052857 0 0.025703 rpy=0 0 0, axis 0 1 0, limit lower=0 upper=0.62 effort=10.43 velocity=1, mimic joint=left_middle_mcp_pitch multiplier=0.46 offset=0
- added joint left_middle_mcp_pitch: type revolute, parent leftHand_link, child left_middle_proximal, origin xyz=-0.0021316 -0.0076542 0.15281 rpy=0 -0.0087266 0, axis 0 1 0, limit lower=0 upper=1.36 effort=4.8 velocity=1
- added joint left_middle_pip: type revolute, parent left_middle_proximal, child left_middle_middle, origin xyz=-0.0010861 0 0.035634 rpy=0 0 0, axis 0 1 0, limit lower=0 upper=1.78 effort=3.7 velocity=1, mimic joint=left_middle_mcp_pitch multiplier=1.3 offset=0
- added joint left_nero_base_mount_joint: type fixed, parent leftArm_link, child left_nero_base_link, origin xyz=0 0 0 rpy=1.5708 0 1.5708
- added joint left_nero_gripper_flange_joint: type fixed, parent left_nero_link7, child left_nero_gripper_flange, origin xyz=0.031 0 -0.0235 rpy=-1.5708 0 -1.5708
- added joint left_nero_joint2: type revolute, parent left_nero_link1, child left_nero_link2, origin xyz=0 0 0 rpy=1.5707963 1.5707963 0, axis 0 0 1, limit lower=-3.3107963 upper=0.1692037 effort=100 velocity=5
- added joint left_nero_joint3: type revolute, parent left_nero_link2, child left_nero_link3, origin xyz=0 -0.31 0 rpy=-1.5707963  0 3.1415926926, axis 0 0 1, limit lower=-2.75 upper=2.75 effort=100 velocity=5
- added joint left_nero_joint4: type revolute, parent left_nero_link3, child left_nero_link4, origin xyz=0 0 0 rpy=-1.5707963  0 3.1415926926, axis 0 0 1, limit lower=-1.01 upper=2.14 effort=100 velocity=5
- added joint left_nero_joint5: type revolute, parent left_nero_link4, child left_nero_link5, origin xyz=0 -0.27001 0 rpy=1.5707963  -1.5707963  0, axis 0 0 1, limit lower=-2.75 upper=2.75 effort=100 velocity=5
- added joint left_nero_joint6: type revolute, parent left_nero_link5, child left_nero_link6, origin xyz=0 0 0 rpy=1.5707963  -1.5707963  0, axis 0 0 1, limit lower=-0.73 upper=0.95 effort=100 velocity=5
- added joint left_nero_joint7: type revolute, parent left_nero_link6, child left_nero_link7, origin xyz=0 -0.0235 0 rpy=1.5707963 0 0, axis 0 0 1, limit lower=-1.5707963 upper=1.5707963 effort=100 velocity=5
- added joint left_pinky_dip: type revolute, parent left_pinky_middle, child left_pinky_distal, origin xyz=-0.0052444 0 0.025711 rpy=0 0 0, axis 0 1 0, limit lower=0 upper=0.62 effort=10.43 velocity=1, mimic joint=left_pinky_mcp_pitch multiplier=0.46 offset=0
- added joint left_pinky_mcp_pitch: type revolute, parent left_pinky_metacarpals, child left_pinky_proximal, origin xyz=0.0022097 0 0.015275 rpy=0 0 0, axis 0 1 0, limit lower=0 upper=1.36 effort=4.8 velocity=1
- added joint left_pinky_mcp_roll: type revolute, parent leftHand_link, child left_pinky_metacarpals, origin xyz=-0.00012074 0.030346 0.12755 rpy=-0.057596 -0.0087266 0, axis -1 0 0, limit lower=0 upper=0.3 effort=4.29 velocity=1
- added joint left_pinky_pip: type revolute, parent left_pinky_proximal, child left_pinky_middle, origin xyz=-0.0010697 0 0.035634 rpy=0 0 0, axis 0 1 0, limit lower=0 upper=1.78 effort=3.7 velocity=1, mimic joint=left_pinky_mcp_pitch multiplier=1.3 offset=0
- added joint left_ring_dip: type revolute, parent left_ring_middle, child left_ring_distal, origin xyz=-0.0052444 0 0.025711 rpy=0 0 0, axis 0 1 0, limit lower=0 upper=0.62 effort=10.43 velocity=1, mimic joint=left_ring_mcp_pitch multiplier=0.46 offset=0
- added joint left_ring_mcp_pitch: type revolute, parent left_ring_metacarpals, child left_ring_proximal, origin xyz=0.0022097 0 0.015275 rpy=0 0 0, axis 0 1 0, limit lower=0 upper=1.36 effort=4.8 velocity=1
- added joint left_ring_mcp_roll: type revolute, parent leftHand_link, child left_ring_metacarpals, origin xyz=-0.0021643 0.011346 0.13253 rpy=-0.024435 -0.0087266 0, axis -1 0 0, limit lower=0 upper=0.2 effort=4.29 velocity=1
- added joint left_ring_pip: type revolute, parent left_ring_proximal, child left_ring_middle, origin xyz=-0.0010697 0 0.035634 rpy=0 0 0, axis 0 1 0, limit lower=0 upper=1.78 effort=3.7 velocity=1, mimic joint=left_ring_mcp_pitch multiplier=1.3 offset=0
- added joint left_thumb_cmc_pitch: type revolute, parent left_thumb_metacarpals_base2, child left_thumb_metacarpals, origin xyz=0.0036974 -0.015398 -0.0019891 rpy=0 -0.9163 1.8064, axis 0 1 0, limit lower=0 upper=0.52 effort=4.8 velocity=1
- added joint left_thumb_cmc_roll: type revolute, parent leftHand_link, child left_thumb_metacarpals_base1, origin xyz=-0.013419 -0.012551 0.060602 rpy=0 0 0, axis -0.99996 0 -0.0087265, limit lower=0 upper=1.03 effort=4.8 velocity=1
- added joint left_thumb_cmc_yaw: type revolute, parent left_thumb_metacarpals_base1, child left_thumb_metacarpals_base2, origin xyz=0.035797 0.00065879 0.00045944 rpy=0.13232 -0.0087266 0, axis 0 0.087156 0.99619, limit lower=0 upper=1.40 effort=4.8 velocity=1
- added joint left_thumb_ip: type revolute, parent left_thumb_proximal, child left_thumb_distal, origin xyz=-0.00017064 0 0.038665 rpy=0 0 0, axis 0 1 0, limit lower=0 upper=0.78 effort=3.36 velocity=1, mimic joint=left_thumb_cmc_pitch multiplier=1.49 offset=0
- added joint left_thumb_mcp: type revolute, parent left_thumb_metacarpals, child left_thumb_proximal, origin xyz=0.0061722 0 0.047968 rpy=0 0 0, axis 0 1 0, limit lower=0 upper=0.72 effort=3.7 velocity=1, mimic joint=left_thumb_cmc_pitch multiplier=1.38 offset=0
- added joint rightArm_base_joint: type fixed, parent waist_link3, child rightArm_link, origin xyz=0.0073775 0.42752 0.1076 rpy=0 0 0
- added joint right_index_dip: type revolute, parent right_index_middle, child right_index_distal, origin xyz=-0.0052444 0 0.025711 rpy=0 0 0, axis 0 1 0, limit lower=0 upper=0.62 effort=10.43 velocity=1, mimic joint=right_index_mcp_pitch multiplier=0.46 offset=0
- added joint right_index_mcp_pitch: type revolute, parent right_index_metacarpals, child right_index_proximal, origin xyz=0.00220968332188026 0 0.0152749792820048 rpy=0 0 0, axis 0 1 0, limit lower=0 upper=1.36 effort=4.8 velocity=1
- added joint right_index_mcp_roll: type revolute, parent rightHand_link, child right_index_metacarpals, origin xyz=-0.0021643 0.026654 0.13253 rpy=-0.027925 -0.0087266 0, axis -1 0 0, limit lower=0 upper=0.19 effort=100 velocity=1
- added joint right_index_pip: type revolute, parent right_index_proximal, child right_index_middle, origin xyz=-0.0010697 0 0.035634 rpy=0 0 0, axis 0 1 0, limit lower=0 upper=1.78 effort=3.7 velocity=1, mimic joint=right_index_mcp_pitch multiplier=1.3 offset=0
- added joint right_middle_dip: type revolute, parent right_middle_middle, child right_middle_distal, origin xyz=-0.0055098 0 0.025656 rpy=0 0 0, axis 0 1 0, limit lower=0 upper=0.62 effort=10.43 velocity=1, mimic joint=right_middle_mcp_pitch multiplier=0.46 offset=0
- added joint right_middle_mcp_pitch: type revolute, parent rightHand_link, child right_middle_proximal, origin xyz=-0.00213155528434806 0.00765417737818821 0.152810108410232 rpy=0 0 0, axis 0 1 0, limit lower=0 upper=1.36 effort=100 velocity=1
- added joint right_middle_pip: type revolute, parent right_middle_proximal, child right_middle_middle, origin xyz=-0.00139702428111229 0 0.0356230829860553 rpy=0 0 0, axis 0 1 0, limit lower=0 upper=1.78 effort=3.7 velocity=1, mimic joint=right_middle_mcp_pitch multiplier=1.3 offset=0
- added joint right_nero_base_mount_joint: type fixed, parent rightArm_link, child right_nero_base_link, origin xyz=0 0 0 rpy=-1.5708 0 1.5708
- added joint right_nero_gripper_flange_joint: type fixed, parent right_nero_link7, child right_nero_gripper_flange, origin xyz=0.031 0 -0.0235 rpy=-1.5708 0 -1.5708
- added joint right_nero_joint2: type revolute, parent right_nero_link1, child right_nero_link2, origin xyz=0 0 0 rpy=1.5707963 1.5707963 0, axis 0 0 1, limit lower=-3.3107963 upper=0.1692037 effort=100 velocity=5
- added joint right_nero_joint3: type revolute, parent right_nero_link2, child right_nero_link3, origin xyz=0 -0.31 0 rpy=-1.5707963  0 3.1415926926, axis 0 0 1, limit lower=-2.75 upper=2.75 effort=100 velocity=5
- added joint right_nero_joint4: type revolute, parent right_nero_link3, child right_nero_link4, origin xyz=0 0 0 rpy=-1.5707963  0 3.1415926926, axis 0 0 1, limit lower=-1.01 upper=2.14 effort=100 velocity=5
- added joint right_nero_joint5: type revolute, parent right_nero_link4, child right_nero_link5, origin xyz=0 -0.27001 0 rpy=1.5707963  -1.5707963  0, axis 0 0 1, limit lower=-2.75 upper=2.75 effort=100 velocity=5
- added joint right_nero_joint6: type revolute, parent right_nero_link5, child right_nero_link6, origin xyz=0 0 0 rpy=1.5707963  -1.5707963  0, axis 0 0 1, limit lower=-0.73 upper=0.95 effort=100 velocity=5
- added joint right_nero_joint7: type revolute, parent right_nero_link6, child right_nero_link7, origin xyz=0 -0.0235 0 rpy=1.5707963 0 0, axis 0 0 1, limit lower=-1.5707963 upper=1.5707963 effort=100 velocity=5
- added joint right_pinky_dip: type revolute, parent right_pinky_middle, child right_pinky_distal, origin xyz=-0.0052444 0 0.025711 rpy=0 0 0, axis 0 1 0, limit lower=0 upper=0.62 effort=10.43 velocity=1, mimic joint=right_pinky_mcp_pitch multiplier=0.46 offset=0
- added joint right_pinky_mcp_pitch: type revolute, parent right_pinky_metacarpals, child right_pinky_proximal, origin xyz=0.0022097 0 0.015275 rpy=0 0 0, axis 0 1 0, limit lower=0 upper=1.36 effort=4.8 velocity=1
- added joint right_pinky_mcp_roll: type revolute, parent rightHand_link, child right_pinky_metacarpals, origin xyz=-0.00012074 -0.030346 0.12755 rpy=0.057596 -0.0087266 0, axis 1 0 0, limit lower=0 upper=0.3 effort=4.29 velocity=1
- added joint right_pinky_pip: type revolute, parent right_pinky_proximal, child right_pinky_middle, origin xyz=-0.0010697 0 0.035634 rpy=0 0 0, axis 0 1 0, limit lower=0 upper=1.78 effort=3.7 velocity=1, mimic joint=right_pinky_mcp_pitch multiplier=1.34 offset=0
- added joint right_ring_dip: type revolute, parent right_ring_middle, child right_ring_distal, origin xyz=-0.00524443259686075 0 0.0257114125710868 rpy=0 0 -0.000213216385347256, axis 0.000213099161087669 0.999450193223668 -0.033155178387707, limit lower=0 upper=0.62 effort=10.43 velocity=1, mimic joint=right_ring_mcp_pitch multiplier=0.46 offset=0
- added joint right_ring_mcp_pitch: type revolute, parent right_ring_metacarpals, child right_ring_proximal, origin xyz=0.0022097 0 0.015275 rpy=0 0 0, axis 0 1 0, limit lower=0 upper=1.36 effort=4.8 velocity=1
- added joint right_ring_mcp_roll: type revolute, parent rightHand_link, child right_ring_metacarpals, origin xyz=-0.00216430029569533 -0.0113458226218121 0.132534071328313 rpy=0.0244346095279086 -0.00872664625996829 0, axis 1 0 0, limit lower=0 upper=0.2 effort=4.29 velocity=1
- added joint right_ring_pip: type revolute, parent right_ring_proximal, child right_ring_middle, origin xyz=-0.00106974956301328 0 0.0356344124989653 rpy=0 0 0, axis 0 1 0, limit lower=0 upper=1.78 effort=3.7 velocity=1, mimic joint=right_ring_mcp_pitch multiplier=1.34 offset=0
- added joint right_thumb_cmc_pitch: type revolute, parent right_thumb_metacarpals_base2, child right_thumb_metacarpals, origin xyz=0.0037151 0.015396 -0.0019302 rpy=0 -0.9163 -1.8076, axis 0 1 0, limit lower=0 upper=0.52 effort=4.8 velocity=1
- added joint right_thumb_cmc_roll: type revolute, parent rightHand_link, child right_thumb_metacarpals_base1, origin xyz=-0.013419 0.012551 0.060602 rpy=0 0 0, axis 0.99996 0 -0.0087265, limit lower=0 upper=1.03 effort=4.8 velocity=1
- added joint right_thumb_cmc_yaw: type revolute, parent right_thumb_metacarpals_base1, child right_thumb_metacarpals_base2, origin xyz=0.035798 -0.0006691 0.00040146 rpy=-0.13233 -0.0085747 0.0011413, axis 0 0 -1, limit lower=0 upper=1.40 effort=4.8 velocity=1
- added joint right_thumb_ip: type revolute, parent right_thumb_proximal, child right_thumb_distal, origin xyz=-0.00017064 0 0.038665 rpy=0 0 0, axis 0 1 0, limit lower=0 upper=0.78 effort=3.36 velocity=1, mimic joint=right_thumb_cmc_pitch multiplier=1.49 offset=0
- added joint right_thumb_mcp: type revolute, parent right_thumb_metacarpals, child right_thumb_proximal, origin xyz=0.0061722 0 0.047968 rpy=0 0 0, axis 0 1 0, limit lower=0 upper=0.72 effort=3.7 velocity=1, mimic joint=right_thumb_cmc_pitch multiplier=1.38 offset=0
- joint leftArm_joint: axis -0.0016361 0 1 -> 0 0 1; child leftArm_link -> left_nero_link1; limit lower=0 upper=3.14 effort=0 velocity=0 -> lower=-2.70526 upper=2.70526 effort=100 velocity=5; origin xyz=0.0076949 0.42752 -0.086398 rpy=0 0 0 -> xyz=0 -0.138 -0.000000506902 rpy=1.5708 0 0; parent waist_link3 -> left_nero_base_link
- joint leftHand_joint: axis 0 0 0 -> (none); origin xyz=-0.00021023 -0.0865 0 rpy=0 0 0 -> xyz=-0.00021023 -0.0865 0 rpy=1.5708 3.1416 0
- joint leftSensor_joint: axis 0 0 0 -> (none); origin xyz=-0.0012639 -0.613 -0.1381 rpy=0 0 0 -> xyz=0 0 0.012 rpy=-1.5708 0 0; parent leftArm_link -> left_nero_gripper_flange
- joint rightArm_joint: axis 0.0016361 0 -1 -> 0 0 1; child rightArm_link -> right_nero_link1; limit lower=0 upper=3.14 effort=0 velocity=0 -> lower=-2.70526 upper=2.70526 effort=100 velocity=5; origin xyz=0.0073775 0.42752 0.1076 rpy=0 0 0 -> xyz=0 -0.138 -0.000000506902 rpy=1.5708 0 0; parent waist_link3 -> right_nero_base_link
- joint rightHand_joint: axis 0 0 0 -> (none); origin xyz=-0.00021023 -0.0865 0 rpy=0 0 0 -> xyz=-0.00021023 -0.0865 0 rpy=1.5708 3.1416 0
- joint rightSensor_joint: axis 0 0 0 -> (none); origin xyz=-0.0017158 -0.613 0.1381 rpy=0 0 0 -> xyz=0 0 0.012 rpy=-1.5708 0 0; parent rightArm_link -> right_nero_gripper_flange
